File: Electronics/Reflow Hot Plate Schematic.kicad_sch (KiCad schematic)
At the start: 9 parts, among them SW1 SW_Push, SW2 SW_Push, U1 SSR-25DA, U2 74HC595, U3 LCD1602, U4 MAX6675

Commit message: Updated temperature sensing
Connections:
- net SO: now reaches A1.17 (D2)
- net SO: now also U4.7 (SO)
- net at A1.26 (D11): no longer U4.7 (SO)
Changed lines of the file:
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@@
-	(wire
-		(pts
-			(xy 109.22 86.36) (xy 119.38 86.36)
-		)
-		(stroke
-			(width 0)
-			(type default)
-		)
-	)
 	(wire
 		(pts
@@
 	(wire
 		(pts
+			(xy 106.68 63.5) (xy 119.38 63.5)
+		)
+		(stroke
+			(width 0)
+			(type default)
+		)
+	)
+	(wire
+		(pts
 			(xy 95.25 102.87) (xy 95.25 104.14)
 		)
@@
 		(pts
 			(xy 165.1 139.7) (xy 177.8 139.7)
-		)
-		(stroke
-			(width 0)
-			(type default)
-		)
-	)
-	(wire
-		(pts
-			(xy 109.22 92.71) (xy 109.22 86.36)
 		)
 		(stroke
@@
 		)
 	)
+	(label "SO"
+		(at 106.68 63.5 0)
+		(effects
+			(font
+				(size 1.27 1.27)
+			)
+			(justify left bottom)
+		)
+	)
 	(label "QG"
 		(at 154.94 130.81 0)
@@
 		)
 	)
+	(label "SO"
+		(at 109.22 92.71 180)
+		(effects
+			(font
+				(size 1.27 1.27)
+			)
+			(justify right bottom)
+		)
+	)

Commit message: Added full GUI and editability of heating parameters
Connections:
- net RCLK: now also A1.25 (D10); no longer A1.19 (D4)
- net SO: now also A1.22 (D7); no longer A1.17 (D2)
- net SRCLK: now also A1.24 (D9); no longer A1.18 (D3)
- net SW_1: no longer A1.15 (D0/RX)
- net SW_2: no longer A1.16 (D1/TX)
- new net SW_DOWN: A1.18 (D3)
- new net SW_NEXT: A1.19 (D4)
- new net SW_UP: A1.17 (D2)
Changed lines of the file:
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@@
-	(wire
-		(pts
-			(xy 106.68 58.42) (xy 119.38 58.42)
-		)
-		(stroke
-			(width 0)
-			(type default)
-		)
-	)
 	(wire
 		(pts
@@
 	(wire
 		(pts
+			(xy 106.68 76.2) (xy 119.38 76.2)
+		)
+		(stroke
+			(width 0)
+			(type default)
+		)
+	)
+	(wire
+		(pts
 			(xy 167.64 68.58) (xy 165.1 68.58)
 		)
@@
 	(wire
 		(pts
+			(xy 106.68 68.58) (xy 119.38 68.58)
+		)
+		(stroke
+			(width 0)
+			(type default)
+		)
+	)
+	(wire
+		(pts
 			(xy 114.3 91.44) (xy 119.38 91.44)
 		)
@@
 	(wire
 		(pts
+			(xy 106.68 83.82) (xy 119.38 83.82)
+		)
+		(stroke
+			(width 0)
+			(type default)
+		)
+	)
+	(wire
+		(pts
 			(xy 95.25 83.82) (xy 95.25 85.09)
 		)
@@
 	(wire
 		(pts
-			(xy 106.68 60.96) (xy 119.38 60.96)
-		)
-		(stroke
-			(width 0)
-			(type default)
-		)
-	)
-	(wire
-		(pts
 			(xy 165.1 120.65) (xy 167.64 120.65)
 		)
@@
 	(wire
 		(pts
+			(xy 106.68 81.28) (xy 119.38 81.28)
+		)
+		(stroke
+			(width 0)
+			(type default)
+		)
+	)
+	(wire
+		(pts
 			(xy 167.64 128.27) (xy 154.94 128.27)
 		)
@@
 	(wire
 		(pts
-			(xy 106.68 68.58) (xy 119.38 68.58)
-		)
-		(stroke
-			(width 0)
-			(type default)
-		)
-	)
-	(wire
-		(pts
 			(xy 165.1 139.7) (xy 177.8 139.7)
 		)
@@
 			(width 0)
 			(type default)
-		)
-	)
-	(label "SRCLK"
-		(at 106.68 66.04 0)
-		(effects
-			(font
-				(size 1.27 1.27)
-			)
-			(justify left bottom)
 		)
 	)
@@
 		)
 	)
-	(label "SO"
-		(at 106.68 63.5 0)
-		(effects
-			(font
-				(size 1.27 1.27)
-			)
-			(justify left bottom)
-		)
-	)
 	(label "QG"
 		(at 154.94 130.81 0)
@@
 		)
 	)
+	(label "SO"
+		(at 106.68 76.2 0)
+		(effects
+			(font
+				(size 1.27 1.27)
+			)
+			(justify left bottom)
+		)
+	)
 	(label "QG"
 		(at 199.39 68.58 180)
@@
 		)
 	)
+	(label "SW_DOWN"
+		(at 106.68 66.04 0)
+		(effects
+			(font
+				(size 1.27 1.27)
+			)
+			(justify left bottom)
+		)
+	)
+	(label "SW_NEXT"
+		(at 106.68 68.58 0)
+		(effects
+			(font
+				(size 1.27 1.27)
+			)
+			(justify left bottom)
+		)
+	)
 	(label "QF"
 		(at 154.94 128.27 0)
@@
 		)
 	)
-	(label "SW_1"
-		(at 106.68 58.42 0)
-		(effects
-			(font
-				(size 1.27 1.27)
-			)
-			(justify left bottom)
-		)
-	)
 	(label "SER"
 		(at 154.94 53.34 0)
@@
 	)
 	(label "SRCLK"
+		(at 106.68 81.28 0)
+		(effects
+			(font
+				(size 1.27 1.27)
+			)
+			(justify left bottom)
+		)
+	)
+	(label "SRCLK"
 		(at 154.94 58.42 0)
 		(effects
@@
 		)
 	)
-	(label "SW_2"
-		(at 106.68 60.96 0)
-		(effects
-			(font
-				(size 1.27 1.27)
-			)
-			(justify left bottom)
-		)
-	)
 	(label "RCLK"
 		(at 154.94 66.04 0)
@@
 		)
 	)
-	(label "RCLK"
-		(at 106.68 68.58 0)
-		(effects
-			(font
-				(size 1.27 1.27)
-			)
-			(justify left bottom)
-		)
-	)
 	(label "E"
 		(at 199.39 60.96 180)
@@
 		(effects
 			(font
+				(size 1.27 1.27)
+			)
+			(justify left bottom)
+		)
+	)
+	(label "RCLK"
+		(at 106.68 83.82 0)
+		(effects
+			(font
+				(size 1.27 1.27)
+			)
+			(justify left bottom)
+		)
+	)
+	(label "SW_UP"
+		(at 106.68 63.5 0)
+		(effects
+			(font

Commit message: Screenshot schematic
Parts:
- added SW3: SW_Push, symbol Switch:SW_Push
Connections:
- net SW_1 is gone; now on net GND: SW1.2
- net SW_2 is gone; now on net SW_DOWN: SW2.2
- net GND: now also SW3.1; no longer SW1.1
- net SW_NEXT: now also SW3.2
- net SW_UP: now also SW1.1
Other:
- moved on the sheet: RV1, SW1, SW2, U3
